Commit message: Correção de pequenos bugs

File: src/robot/kinect/kinect_v2.urdf.xacro (robot description, xacro)
@@ -19,5 +19,5 @@
                 <origin xyz="0 0 0" rpy="0 0 0" />
                 <geometry>
-                    <mesh filename="$(find p3dxbot)/robot/kinect/meshes/kinect2.STL" />
+                    <mesh filename="package://p3dxbot/robot/kinect/meshes/kinect2.STL" />
                 </geometry>
                 <material name="">
@@ -28,5 +28,5 @@
                 <origin xyz="0 0 0" rpy="0 0 0" />
                 <geometry>
-                    <mesh filename="$(find p3dxbot)/robot/kinect/meshes/kinect2.STL" />
+                    <mesh filename="package://p3dxbot/robot/kinect/meshes/kinect2.STL" />
                 </geometry>
             </collision>

File: src/urdf/pioneer3dxAtividade.xacro (robot description, xacro)
@@ -6,5 +6,5 @@
   <!-- Import robot -->
   <xacro:include filename="$(find p3dxbot)/robot/pioneer3dx_body.xacro"/>
-  <xacro:pioneer3dx_body name="chassis" parent="base_link" meshes="$(find p3dxbot)/robot/meshes/p3dx"/>
+  <xacro:pioneer3dx_body name="chassis" parent="base_link" meshes="package://p3dxbot/robot/meshes/p3dx"/>
   <!-- Import Kinect -->
 <xacro:include filename="$(find p3dxbot)/robot/kinect/kinect_v2.urdf.xacro" />
